Commit message: feat: visualize livox mesh model

File: urdf/mid360.xacro (robot description, xacro)
@@ -24,5 +24,5 @@
   <visual>
         <geometry>
-            <box size="${length} ${width} ${height}"/>
+            <mesh filename="package://ros2_livox_simulation/meshes/mid-360-scaled.dae" scale="1.0 1.0 1.0"/>
         </geometry>
   </visual>
